File: PCB/Main Boards/OSO-SWAT-A1-04.brd (EAGLE design)
At the start: 24.4 x 24.4 mm, 36 parts, among them J1 FH19C-9S-0.5SH_10_, U1 ATSAML22J18A-MUT, U2 MIC5365-3.3YC5-TR

Commit message: rename segments in schematic to match SLCD driver
Connections:
- net SEG24 renamed SEG15
- net SEG25 renamed SEG14
- net SEG26 renamed SEG13
- net SEG27 renamed SEG12
- net SEG28 renamed SEG11
- net SEG0: now also U$2.27, U1.12; no longer U$2.17, U1.25
- net SEG1: now also U$2.26, U1.13; no longer U$2.18, U1.24
- net SEG10: now also U$2.17, U1.25; no longer U$2.27, U1.12
- net SEG16: now also U$2.11, U1.31; no longer U$2.1, U1.40
- net SEG17: now also U$2.10, U1.32; no longer U$2.2, U1.39
- net SEG18: now also U$2.6, U1.35; no longer U$2.3, U1.38
- net SEG19: now also U$2.5, U1.36; no longer U$2.4, U1.37
- net SEG2: now also U$2.25, U1.14; no longer U$2.19, U1.20
- net SEG20: now also U$2.4, U1.37; no longer U$2.5, U1.36
- net SEG21: now also U$2.3, U1.38; no longer U$2.6, U1.35
- net SEG22: now also U$2.2, U1.39; no longer U$2.10, U1.32
- net SEG23: now also U$2.1, U1.40; no longer U$2.11, U1.31
- net SEG3: now also U$2.24, U1.15; no longer U$2.20, U1.19
- net SEG4: now also U$2.23, U1.16; no longer U$2.21, U1.18
- net SEG6: now also U$2.21, U1.18; no longer U$2.23, U1.16
- net SEG7: now also U$2.20, U1.19; no longer U$2.24, U1.15
- net SEG8: now also U$2.19, U1.20; no longer U$2.25, U1.14
- net SEG9: now also U$2.18, U1.24; no longer U$2.26, U1.13
Routing:
- net SEG23: track 3.51 -> 10.6 mm
- net SEG16: track 10.6 -> 3.51 mm
- net SEG22: track 3.90 -> 9.72 mm
- net SEG17: track 9.72 -> 3.90 mm
- net SEG10: track 7.76 -> 4.01 mm
- net SEG0: track 4.01 -> 7.76 mm
- net SEG9: track 6.98 -> 4.22 mm
- net SEG1: track 4.22 -> 6.98 mm
- net SEG8: track 6.20 -> 3.62 mm
- net SEG2: track 3.62 -> 6.20 mm
- net SEG21: track 6.28 -> 8.74 mm
- net SEG18: track 8.74 -> 6.28 mm
- net SEG6: track 4.65 -> 6.31 mm
- net SEG4: track 6.31 -> 4.65 mm
- net SEG7: track 5.41 -> 3.95 mm
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Changed lines of the file:
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@@
 <wire x1="-3.2135" y1="7.2005" x2="5.8367625" y2="7.2005" width="0.127" layer="1"/>
 </signal>
-<signal name="SEG16">
+<signal name="SEG23">
 <contactref element="U$2" pad="1"/>
 <contactref element="U1" pad="40"/>
@@
 <wire x1="-9.148" y1="5.6039875" x2="-8.255" y2="4.7109875" width="0.127" layer="1"/>
 </signal>
-<signal name="SEG17">
+<signal name="SEG22">
 <contactref element="U$2" pad="2"/>
 <contactref element="U1" pad="39"/>
@@
 <wire x1="-8.442" y1="5.5112" x2="-7.8957875" y2="4.9649875" width="0.127" layer="1"/>
 </signal>
-<signal name="SEG18">
+<signal name="SEG21">
 <contactref element="U$2" pad="3"/>
 <contactref element="U1" pad="38"/>
@@
 <wire x1="-7.736" y1="5.45" x2="-7.62" y2="5.334" width="0.127" layer="1"/>
 </signal>
-<signal name="SEG19">
+<signal name="SEG20">
 <contactref element="U$2" pad="4"/>
 <contactref element="U1" pad="37"/>
@@
 <wire x1="-5.433" y1="0.5689" x2="-4.0132" y2="0.5689" width="0.127" layer="1"/>
 </signal>
-<signal name="SEG20">
+<signal name="SEG19">
 <contactref element="U$2" pad="5"/>
 <contactref element="U1" pad="36"/>
@@
 <wire x1="-4.0132" y1="1.0689" x2="-5.425" y2="1.0689" width="0.127" layer="1"/>
 </signal>
-<signal name="SEG21">
+<signal name="SEG18">
 <contactref element="U$2" pad="6"/>
 <contactref element="U1" pad="35"/>
@@
 <wire x1="-5.6261" y1="4.7625" x2="-5.6261" y2="1.7907" width="0.127" layer="1"/>
 </signal>
-<signal name="SEG22">
+<signal name="SEG17">
 <contactref element="U$2" pad="10"/>
 <contactref element="U1" pad="32"/>
@@
 <wire x1="-2.3368" y1="5.2781875" x2="-2.3368" y2="4.29410625" width="0.127" layer="1"/>
 </signal>
-<signal name="SEG23">
+<signal name="SEG16">
 <contactref element="U$2" pad="11"/>
 <contactref element="U1" pad="31"/>
@@
 <wire x1="-2.44790625" y1="3.81" x2="-1.991709375" y2="4.266196875" width="0.127" layer="1"/>
 </signal>
-<signal name="SEG0">
+<signal name="SEG10">
 <contactref element="U$2" pad="17"/>
 <contactref element="U1" pad="25"/>
@@
 <wire x1="1.894" y1="5.207" x2="1.651" y2="5.207" width="0.127" layer="1"/>
 </signal>
-<signal name="SEG2">
+<signal name="SEG8">
 <contactref element="U$2" pad="19"/>
 <contactref element="U1" pad="20"/>
@@
 <wire x1="3.06078125" y1="5.3022" x2="2.7326" y2="4.97401875" width="0.127" layer="1"/>
 </signal>
-<signal name="SEG3">
+<signal name="SEG7">
 <contactref element="U$2" pad="20"/>
 <contactref element="U1" pad="19"/>
@@
 <wire x1="4.266" y1="5.5804" x2="4.266" y2="6.25" width="0.127" layer="1"/>
 </signal>
-<signal name="SEG4">
+<signal name="SEG6">
 <contactref element="U$2" pad="21"/>
 <contactref element="U1" pad="18"/>
@@
 <wire x1="5.2451" y1="2.9083" x2="6.115" y2="3.7782" width="0.127" layer="1"/>
 </signal>
-<signal name="SEG6">
+<signal name="SEG4">
 <contactref element="U$2" pad="23"/>
 <contactref element="U1" pad="16"/>
@@
 <wire x1="6.384" y1="3.6698125" x2="6.384" y2="6.25" width="0.127" layer="1"/>
 </signal>
-<signal name="SEG7">
+<signal name="SEG3">
 <contactref element="U$2" pad="24"/>
 <contactref element="U1" pad="15"/>
@@
 <wire x1="5.2439" y1="2.0689" x2="7.09" y2="3.915" width="0.127" layer="1"/>
 </signal>
-<signal name="SEG8">
+<signal name="SEG2">
 <contactref element="U$2" pad="25"/>
 <contactref element="U1" pad="14"/>
@@
 <wire x1="5.2301125" y1="1.5689" x2="7.796" y2="4.1347875" width="0.127" layer="1"/>
 </signal>
-<signal name="SEG9">
+<signal name="SEG1">
 <contactref element="U$2" pad="26"/>
 <contactref element="U1" pad="13"/>
@@
 <wire x1="8.502" y1="4.354575" x2="8.502" y2="6.25" width="0.127" layer="1"/>
 </signal>
-<signal name="SEG10">
+<signal name="SEG0">
 <contactref element="U$2" pad="27"/>
 <wire x1="9.208" y1="4.58934375" x2="9.208" y2="6.25" width="0.127" layer="1"/>
@@
 <wire x1="-0.97911875" y1="-7.2517" x2="-3.1428" y2="-9.41538125" width="0.254" layer="16"/>
 </signal>
-<signal name="SEG24">
+<signal name="SEG15">
 <contactref element="U$2" pad="12"/>
 <contactref element="U1" pad="30"/>
@@
 <wire x1="-1.382" y1="4.502909375" x2="-2.369" y2="3.51590625" width="0.127" layer="1"/>
 </signal>
-<signal name="SEG25">
+<signal name="SEG14">
 <contactref element="U$2" pad="13"/>
 <contactref element="U1" pad="29"/>
@@
 <wire x1="-0.676" y1="4.83590625" x2="-0.676" y2="6.25" width="0.127" layer="1"/>
 </signal>
-<signal name="SEG26">
+<signal name="SEG13">
 <contactref element="U$2" pad="14"/>
 <contactref element="U1" pad="28"/>
@@
 <wire x1="-1.369" y1="3.64290625" x2="0.03" y2="5.04190625" width="0.127" layer="1"/>
 </signal>
-<signal name="SEG27">
+<signal name="SEG12">
 <contactref element="U$2" pad="15"/>
 <contactref element="U1" pad="27"/>
@@
 <wire x1="-0.869" y1="3.703" x2="0.736" y2="5.308003125" width="0.127" layer="1"/>
 </signal>
-<signal name="SEG28">
+<signal name="SEG11">
 <contactref element="U$2" pad="16"/>
 <contactref element="U1" pad="26"/>
@@
 <wire x1="-0.369" y1="3.64290625" x2="1.442" y2="5.45390625" width="0.127" layer="1"/>
 </signal>
-<signal name="SEG1">
+<signal name="SEG9">
 <contactref element="U$2" pad="18"/>
 <contactref element="U1" pad="24"/>

Commit message: fix LED part number, make boards identical
Parts:
- LED: value QBLP655R -> QBLP655-RIG; device QBLP655R:LED_QBLP655R -> QBLP655:LED_QBLP655
Changed lines of the file:
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@@
 <attribute name="VALUE" x="6.33821875" y="-14.05451875" size="0.508" layer="28" font="vector" ratio="18" rot="MR0" align="center"/>
-</element>
-<element name="LED" library="QBLP655R" package="LED_QBLP655R" value="QBLP655R" x="-11.3284" y="0" smashed="yes" rot="R90">
-<attribute name="DESCRIPTION" value=" Green, Red 571nm Green, 631nm Red LED Indication - Discrete 2V Green, 2V Red 1206 (3216 Metric) " x="-11.3284" y="0" size="0.508" layer="27" font="vector" ratio="18" rot="R90" display="off"/>
-<attribute name="DIGI-KEY_PART_NUMBER" value="160-2026-1-ND" x="-11.3284" y="0" size="0.508" layer="27" font="vector" ratio="18" rot="R90" display="off"/>
-<attribute name="MF" value="Lite-On Inc." x="-11.3284" y="0" size="0.508" layer="27" font="vector" ratio="18" rot="R90" display="off"/>
-<attribute name="MP" value="LTST-C235KGKRKT" x="-11.3284" y="0" size="0.508" layer="27" font="vector" ratio="18" rot="R90" display="off"/>
-<attribute name="NAME" x="-11.340009375" y="0.01056875" size="0.508" layer="25" font="vector" ratio="18" rot="R180" align="center"/>
-<attribute name="PACKAGE" value="1206 Lite-On" x="-11.3284" y="0" size="0.508" layer="27" font="vector" ratio="18" rot="R90" display="off"/>
-<attribute name="PURCHASE-URL" value="https://pricing.snapeda.com/search/part/LTST-C235KGKRKT/?ref=eda" x="-11.3284" y="0" size="0.508" layer="27" font="vector" ratio="18" rot="R90" display="off"/>
-<attribute name="VALUE" x="-9.74758125" y="-0.05493125" size="0.826140625" layer="27" font="vector" ratio="18" rot="R90" align="center"/>
 </element>
 <element name="R8" library="microbuilder" package="_0603MP" value="1K" x="-8.255" y="2.9464" smashed="yes" rot="R180">
@@
 <attribute name="BOM" value="EXCLUDE" x="6.604" y="-9.906" size="1.778" layer="28" rot="MR0" display="off"/>
 <attribute name="REV" value="A" x="6.604" y="-9.906" size="1.778" layer="28" rot="MR0" display="off"/>
+</element>
+<element name="LED" library="QBLP655" package="LED_QBLP655" value="QBLP655-RIG" x="-11.3284" y="0" smashed="yes" rot="R90">
+<attribute name="DESCRIPTION" value=" Green, Red 571nm Green, 631nm Red LED Indication - Discrete 2V Green, 2V Red 1206 (3216 Metric) " x="-11.3284" y="0" size="1.778" layer="27" rot="R90" display="off"/>
+<attribute name="DIGI-KEY_PART_NUMBER" value="160-2026-1-ND" x="-11.3284" y="0" size="1.778" layer="27" rot="R90" display="off"/>
+<attribute name="MF" value="Lite-On Inc." x="-11.3284" y="0" size="1.778" layer="27" rot="R90" display="off"/>
+<attribute name="MP" value="LTST-C235KGKRKT" x="-11.3284" y="0" size="1.778" layer="27" rot="R90" display="off"/>
+<attribute name="NAME" x="-11.340009375" y="0.01056875" size="0.508" layer="25" font="vector" ratio="18" align="center"/>
+<attribute name="PACKAGE" value="1206 Lite-On" x="-11.3284" y="0" size="1.778" layer="27" rot="R90" display="off"/>
+<attribute name="PURCHASE-URL" value="https://pricing.snapeda.com/search/part/LTST-C235KGKRKT/?ref=eda" x="-11.3284" y="0" size="1.778" layer="27" rot="R90" display="off"/>
+<attribute name="VALUE" x="-9.74758125" y="-0.05493125" size="0.826140625" layer="27" font="vector" ratio="18" rot="R90" align="center"/>
 </element>
 </elements>
@@
 <wire x1="-7.6604375" y1="0.0071875" x2="-10.7116125" y2="0.0071875" width="0.127" layer="16"/>
 <via x="-10.922" y="-0.2032" extent="1-16" drill="0.3048"/>
-<contactref element="LED" pad="3"/>
 <wire x1="-10.9284" y1="-1.5" x2="-10.9284" y2="-0.2096" width="0.127" layer="1"/>
 <wire x1="-10.9284" y1="-0.2096" x2="-10.922" y2="-0.2032" width="0.127" layer="1"/>
+<contactref element="LED" pad="3"/>
 </signal>
 <signal name="COM0">
@@
 <wire x1="-7.248425" y1="0.269975" x2="-7.248425" y2="0.2714" width="0.127" layer="16"/>
 <via x="-11.684" y="-0.1096" extent="1-16" drill="0.3048"/>
-<contactref element="LED" pad="1"/>
 <wire x1="-11.7284" y1="-1.5" x2="-11.7284" y2="-0.154" width="0.127" layer="1"/>
 <wire x1="-11.7284" y1="-0.154" x2="-11.684" y2="-0.1096" width="0.127" layer="1"/>
+<contactref element="LED" pad="1"/>
 </signal>
 <signal name="N$1">
 <contactref element="R8" pad="2"/>
-<contactref element="LED" pad="4"/>
 <wire x1="-10.9284" y1="1.5" x2="-10.9284" y2="2.68860625" width="0.127" layer="1"/>
 <wire x1="-9.017" y1="2.9464" x2="-9.3472" y2="3.2766" width="0.127" layer="1"/>
 <wire x1="-10.34040625" y1="3.2766" x2="-9.3472" y2="3.2766" width="0.127" layer="1"/>
 <wire x1="-10.9284" y1="2.68860625" x2="-10.34040625" y2="3.2766" width="0.127" layer="1"/>
+<contactref element="LED" pad="4"/>
 </signal>
 <signal name="N$2">
 <contactref element="R9" pad="2"/>
-<contactref element="LED" pad="2"/>
 <wire x1="-11.7284" y1="1.5" x2="-11.7284" y2="2.267" width="0.127" layer="1"/>
 <wire x1="-10.0076" y1="3.9878" x2="-9.2964" y2="3.9878" width="0.127" layer="1"/>
 <wire x1="-11.7284" y1="2.267" x2="-10.0076" y2="3.9878" width="0.127" layer="1"/>
+<contactref element="LED" pad="2"/>
 </signal>
 <signal name="VBUS_DET">
