File: PCB/Main Boards/OSO-SWAT-A1-04-BLUE.sch (EAGLE design)
At the start: 34 parts, among them J1 FH19C-9S-0.5SH_10_, U1 ATSAML22J18A-MUT, U2 MIC5365-3.3YC5-TR

Commit message: tweak resistor values, move board origin to 0,0
Parts:
- C7, C8: value TBD -> 10pf
- R8: value 100 -> 220
- R9: value 1K -> 220
- X1: value (none) -> 32.768
Changed lines of the file:
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@@
 <part name="C5" library="microbuilder" deviceset="CAP_CERAMIC" device="_0603MP" value="1uF"/>
 <part name="GND14" library="supply1" deviceset="GND" device=""/>
-<part name="X1" library="adafruit" deviceset="XTAL" device="-3.2X1.5"/>
+<part name="X1" library="adafruit" deviceset="XTAL" device="-3.2X1.5" value="32.768"/>
 <part name="C6" library="microbuilder" deviceset="CAP_CERAMIC" device="_0603MP" value="1uF"/>
 <part name="GND2" library="supply1" deviceset="GND" device=""/>
@@
 <part name="RESET" library="EVP-BB1AAB000" deviceset="EVP-BB1AAB000" device=""/>
 <part name="GND15" library="supply1" deviceset="GND" device=""/>
-<part name="R8" library="microbuilder" deviceset="RESISTOR" device="_0603MP" value="100"/>
-<part name="R9" library="microbuilder" deviceset="RESISTOR" device="_0603MP" value="1K"/>
+<part name="R8" library="microbuilder" deviceset="RESISTOR" device="_0603MP" value="220"/>
+<part name="R9" library="microbuilder" deviceset="RESISTOR" device="_0603MP" value="220"/>
 <part name="R2" library="microbuilder" deviceset="RESISTOR" device="_0603MP" value="10K"/>
 <part name="SUPPLY5" library="SparkFun-PowerSymbols" deviceset="VCC" device=""/>
 <part name="R5" library="microbuilder" deviceset="RESISTOR" device="_0603MP" value="10K"/>
-<part name="C7" library="microbuilder" deviceset="CAP_CERAMIC" device="_0402MP" value="TBD"/>
-<part name="C8" library="microbuilder" deviceset="CAP_CERAMIC" device="_0402MP" value="TBD"/>
+<part name="C7" library="microbuilder" deviceset="CAP_CERAMIC" device="_0402MP" value="10pf"/>
+<part name="C8" library="microbuilder" deviceset="CAP_CERAMIC" device="_0402MP" value="10pf"/>
 <part name="U$3" library="microbuilder" deviceset="GND" device=""/>
 <part name="U$9" library="microbuilder" deviceset="GND" device=""/>
