File: PCB/Main Boards/OSO-SWAT-A1-05-BLUE.brd (EAGLE design)
At the start: 24.4 x 24.4 mm, 36 parts, among them J1 FH19C-9S-0.5SH_10_, U1 ATSAML22J18A-MUT, U2 MIC5365-3.3YC5-TR, X1 32.768

Commit message: fix LED resistor values
Parts:
- R8, R9: value 220 -> 100
Changed lines of the file:
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@@
 <drawing>
 <settings>
-<setting alwaysvectorfont="yes"/>
+<setting alwaysvectorfont="no"/>
 <setting keepoldvectorfont="yes"/>
 <setting verticaltext="up"/>
@@
 <attribute name="VALUE" x="18.53021875" y="-1.86251875" size="0.508" layer="28" font="vector" ratio="18" rot="MR0" align="center"/>
 </element>
-<element name="R8" library="microbuilder" package="_0603MP" value="220" x="3.937" y="15.1384" smashed="yes" rot="R180">
+<element name="R8" library="microbuilder" package="_0603MP" value="100" x="3.937" y="15.1384" smashed="yes" rot="R180">
 <attribute name="NAME" x="5.7277" y="15.1384" size="0.508" layer="25" font="vector" ratio="18" rot="R180" align="center"/>
 <attribute name="VALUE" x="4.8895" y="16.0909" size="0.4064" layer="27" ratio="10" rot="R180"/>
 </element>
-<element name="R9" library="microbuilder" package="_0603MP" value="220" x="3.6576" y="16.1798" smashed="yes" rot="R180">
+<element name="R9" library="microbuilder" package="_0603MP" value="100" x="3.6576" y="16.1798" smashed="yes" rot="R180">
 <attribute name="NAME" x="5.4737" y="16.1798" size="0.508" layer="25" font="vector" ratio="18" rot="R180" align="center"/>
 <attribute name="VALUE" x="4.6101" y="17.1323" size="0.4064" layer="27" ratio="10" rot="R180"/>
