File: PCB/Sensor Boards/OSO-MISC-21-021 Sensor Watch Motion II.sch (EAGLE design)
At the start: 8 parts, among them U2 LIS2DW12TR

Commit message: tweaks to the next pair of sensor boards
Parts:
- C1: value 10µF -> 0.1uF
- C2: value 0.1uF -> 10uF
Changed lines of the file:
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@@
 <part name="FRAME1" library="My Stuff" deviceset="A4L-LOC" device=""/>
 <part name="U$3" library="FH19C-9S-0.5SH" deviceset="FH19C-9S-0.5SH_10-FFC" device=""/>
-<part name="C2" library="microbuilder" deviceset="CAP_CERAMIC" device="_0603MP" value="0.1uF"/>
-<part name="C1" library="microbuilder" deviceset="CAP_CERAMIC" device="_0603MP" value="10µF"/>
+<part name="C2" library="microbuilder" deviceset="CAP_CERAMIC" device="_0603MP" value="10uF"/>
+<part name="C1" library="microbuilder" deviceset="CAP_CERAMIC" device="_0603MP" value="0.1uF"/>
 <part name="U$14" library="microbuilder" deviceset="GND" device=""/>
 <part name="U$2" library="microbuilder" deviceset="GND" device=""/>
